File: LSM6DSV320X.kicad_sch (KiCad schematic)
At the start: 1 part, among them U1 LSM6DSV320XTR

Commit message: Revert "Temporary save if I accidentally bust something"
This reverts commit 974f20a02fde00668d4b3d45f60811623d130148.
Parts:
- removed U1: LSM6DSV320XTR, Condor_Imported_Footprints:LGA-14L_2p5X3X0p83_STM, symbol Condor_Imported_Symbols:LSM6DSV320XTR
Changed lines of the file:
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@@
 	(generator_version "10.0")
 	(paper "A4")
-	(symbol
-		(lib_id "Condor_Imported_Symbols:LSM6DSV320XTR")
-		(at 105.41 78.74 0)
-		(unit 1)
-		(body_style 1)
-		(exclude_from_sim no)
-		(in_bom yes)
-		(on_board yes)
-		(in_pos_files yes)
-		(dnp no)
-		(fields_autoplaced yes)
-		(property "Reference" "U1"
-			(at 130.81 66.04 0)
-			(show_name no)
-			(do_not_autoplace no)
-			(effects
-				(font
-					(size 1.524 1.524)
-				)
-			)
-		)
-		(property "Value" "LSM6DSV320XTR"
-			(at 130.81 68.58 0)
-			(show_name no)
-			(do_not_autoplace no)
-			(effects
-				(font
-					(size 1.524 1.524)
-				)
-			)
-		)
-		(property "Footprint" "Condor_Imported_Footprints:LGA-14L_2p5X3X0p83_STM"
-			(at 105.41 78.74 0)
-			(hide yes)
-			(show_name no)
-			(do_not_autoplace no)
-			(effects
-				(font
-					(size 1.27 1.27)
-					(italic yes)
-				)
-			)
-		)
-		(property "Datasheet" "https://www.st.com/resource/en/datasheet/lsm6dsv320x.pdf"
-			(at 105.41 78.74 0)
-			(hide yes)
-			(show_name no)
-			(do_not_autoplace no)
-			(effects
-				(font
-					(size 1.27 1.27)
-					(italic yes)
-				)
-			)
-		)
-		(property "Description" ""
-			(at 105.41 78.74 0)
-			(hide yes)
-			(show_name no)
-			(do_not_autoplace no)
-			(effects
-				(font
-					(size 1.27 1.27)
-				)
-			)
-		)
-		(pin "1"
-		)
-		(pin "2"
-		)
-		(pin "3"
-		)
-		(pin "9"
-		)
-		(pin "6"
-		)
-		(pin "10"
-		)
-		(pin "5"
-		)
-		(pin "4"
-		)
-		(pin "7"
-		)
-		(pin "13"
-		)
-		(pin "11"
-		)
-		(pin "8"
-		)
-		(pin "12"
-		)
-		(pin "14"
-		)
-		(instances
-			(project "Condor"
-				(path "/4a4947c5-540a-4852-b2fa-01bf36e5263c/0a2ef9d1-01fa-4ebe-bda6-b281c88e5853"
-					(reference "U1")
-					(unit 1)
-				)
-			)
-		)
-	)
 )

Commit message: Temporary save if I accidentally bust something
Parts:
- added U1: LSM6DSV320XTR, Condor_Imported_Footprints:LGA-14L_2p5X3X0p83_STM, symbol Condor_Imported_Symbols:LSM6DSV320XTR
Changed lines of the file:
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@@
 	(generator_version "10.0")
 	(paper "A4")
+	(symbol
+		(lib_id "Condor_Imported_Symbols:LSM6DSV320XTR")
+		(at 105.41 78.74 0)
+		(unit 1)
+		(body_style 1)
+		(exclude_from_sim no)
+		(in_bom yes)
+		(on_board yes)
+		(in_pos_files yes)
+		(dnp no)
+		(fields_autoplaced yes)
+		(property "Reference" "U1"
+			(at 130.81 66.04 0)
+			(show_name no)
+			(do_not_autoplace no)
+			(effects
+				(font
+					(size 1.524 1.524)
+				)
+			)
+		)
+		(property "Value" "LSM6DSV320XTR"
+			(at 130.81 68.58 0)
+			(show_name no)
+			(do_not_autoplace no)
+			(effects
+				(font
+					(size 1.524 1.524)
+				)
+			)
+		)
+		(property "Footprint" "Condor_Imported_Footprints:LGA-14L_2p5X3X0p83_STM"
+			(at 105.41 78.74 0)
+			(hide yes)
+			(show_name no)
+			(do_not_autoplace no)
+			(effects
+				(font
+					(size 1.27 1.27)
+					(italic yes)
+				)
+			)
+		)
+		(property "Datasheet" "https://www.st.com/resource/en/datasheet/lsm6dsv320x.pdf"
+			(at 105.41 78.74 0)
+			(hide yes)
+			(show_name no)
+			(do_not_autoplace no)
+			(effects
+				(font
+					(size 1.27 1.27)
+					(italic yes)
+				)
+			)
+		)
+		(property "Description" ""
+			(at 105.41 78.74 0)
+			(hide yes)
+			(show_name no)
+			(do_not_autoplace no)
+			(effects
+				(font
+					(size 1.27 1.27)
+				)
+			)
+		)
+		(pin "1"
+		)
+		(pin "2"
+		)
+		(pin "3"
+		)
+		(pin "9"
+		)
+		(pin "6"
+		)
+		(pin "10"
+		)
+		(pin "5"
+		)
+		(pin "4"
+		)
+		(pin "7"
+		)
+		(pin "13"
+		)
+		(pin "11"
+		)
+		(pin "8"
+		)
+		(pin "12"
+		)
+		(pin "14"
+		)
+		(instances
+			(project "Condor"
+				(path "/4a4947c5-540a-4852-b2fa-01bf36e5263c/0a2ef9d1-01fa-4ebe-bda6-b281c88e5853"
+					(reference "U1")
+					(unit 1)
+				)
+			)
+		)
+	)
 )
