File: Condor.kicad_sch (KiCad schematic)
At the start: 0 parts

Commit message: Multi-page schematic, pulling circuits from Kingfisher, .gitignore
Other:
- added sheet ADXL375 (ADXL375.kicad_sch)
- added sheet BMI088 (BMI088.kicad_sch)
- added sheet Barometer (Barometer.kicad_sch)
- added sheet Charging (Charging.kicad_sch)
- added sheet GPS (GPS.kicad_sch)
- added sheet LSM6DSV320X (LSM6DSV320X.kicad_sch)
- added sheet MCU (MCU.kicad_sch)
- added sheet Magnetometer (Magnetometer.kicad_sch)
- added sheet Memory (Memory.kicad_sch)
- added sheet Power (Power.kicad_sch)
- added sheet USB-C (USB-C.kicad_sch)
- title: (none) -> Condor

Commit message: Reorganizing + importing a few symbols
Other:
- sheet ADXL375: file ADXL375.kicad_sch -> schematics/ADXL375.kicad_sch
- sheet BMI088: file BMI088.kicad_sch -> schematics/BMI088.kicad_sch
- sheet Barometer: file Barometer.kicad_sch -> schematics/Barometer.kicad_sch
- sheet Charging: file Charging.kicad_sch -> schematics/Charging.kicad_sch
- sheet GPS: file GPS.kicad_sch -> schematics/GPS.kicad_sch
- sheet LSM6DSV320X: file LSM6DSV320X.kicad_sch -> schematics/LSM6DSV320X.kicad_sch
- sheet MCU: file MCU.kicad_sch -> schematics/MCU.kicad_sch
- sheet Magnetometer: file Magnetometer.kicad_sch -> schematics/Magnetometer.kicad_sch
- sheet Memory: file Memory.kicad_sch -> schematics/Memory.kicad_sch
- sheet Power: file Power.kicad_sch -> schematics/Power.kicad_sch
- sheet USB-C: file USB-C.kicad_sch -> schematics/USB-C.kicad_sch
Changed lines of the file:
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@@
 			)
 		)
-		(property "Sheetfile" "USB-C.kicad_sch"
+		(property "Sheetfile" "schematics/USB-C.kicad_sch"
 			(at 63.5 169.4946 0)
 			(show_name no)
@@
 			)
 		)
-		(property "Sheetfile" "LSM6DSV320X.kicad_sch"
+		(property "Sheetfile" "schematics/LSM6DSV320X.kicad_sch"
 			(at 17.78 42.4946 0)
 			(show_name no)
@@
 			)
 		)
-		(property "Sheetfile" "Power.kicad_sch"
+		(property "Sheetfile" "schematics/Power.kicad_sch"
 			(at 109.22 137.7446 0)
 			(show_name no)
@@
 			)
 		)
-		(property "Sheetfile" "GPS.kicad_sch"
+		(property "Sheetfile" "schematics/GPS.kicad_sch"
 			(at 154.94 42.4946 0)
 			(show_name no)
@@
 			)
 		)
-		(property "Sheetfile" "Memory.kicad_sch"
+		(property "Sheetfile" "schematics/Memory.kicad_sch"
 			(at 154.94 105.9946 0)
 			(show_name no)
@@
 			)
 		)
-		(property "Sheetfile" "MCU.kicad_sch"
+		(property "Sheetfile" "schematics/MCU.kicad_sch"
 			(at 63.5 105.9946 0)
 			(show_name no)
@@
 			)
 		)
-		(property "Sheetfile" "Barometer.kicad_sch"
+		(property "Sheetfile" "schematics/Barometer.kicad_sch"
 			(at 17.78 137.7446 0)
 			(show_name no)
@@
 			)
 		)
-		(property "Sheetfile" "BMI088.kicad_sch"
+		(property "Sheetfile" "schematics/BMI088.kicad_sch"
 			(at 17.78 105.9946 0)
 			(show_name no)
@@
 			)
 		)
-		(property "Sheetfile" "Magnetometer.kicad_sch"
+		(property "Sheetfile" "schematics/Magnetometer.kicad_sch"
 			(at 17.78 169.4946 0)
 			(show_name no)
@@
 			)
 		)
-		(property "Sheetfile" "ADXL375.kicad_sch"
+		(property "Sheetfile" "schematics/ADXL375.kicad_sch"
 			(at 17.78 74.2446 0)
 			(show_name no)
@@
 			)
 		)
-		(property "Sheetfile" "Charging.kicad_sch"
+		(property "Sheetfile" "schematics/Charging.kicad_sch"
 			(at 63.5 137.7446 0)
 			(show_name no)

Commit message: condor setup
Other:
- sheet ADXL375 renamed IMU ADXL375
- sheet BMI088 renamed IMU BMI088
- sheet LSM6DSV320X renamed IMU LSM6DSV320X
- sheet Memory renamed Storage
- sheet USB-C renamed USB
- removed sheet Charging
- added sheet Pyros (schematics/pyros_condor.kicad_sch)
- sheet Barometer: file schematics/Barometer.kicad_sch -> schematics/barometer_condor.kicad_sch
- sheet GPS: file schematics/GPS.kicad_sch -> schematics/gps_condor.kicad_sch
- sheet IMU ADXL375: file schematics/ADXL375.kicad_sch -> schematics/imu_ADXL375_condor.kicad_sch
- sheet IMU BMI088: file schematics/BMI088.kicad_sch -> schematics/imu_BMI088_condor.kicad_sch
- sheet IMU LSM6DSV320X: file schematics/LSM6DSV320X.kicad_sch -> schematics/imu_LSM6DSV320X_condor.kicad_sch
- sheet MCU: file schematics/MCU.kicad_sch -> schematics/mcu_condor.kicad_sch
- sheet Magnetometer: file schematics/Magnetometer.kicad_sch -> schematics/magnetometer_condor.kicad_sch
- sheet Power: file schematics/Power.kicad_sch -> schematics/power_condor.kicad_sch
- sheet Storage: file schematics/Memory.kicad_sch -> schematics/storage_condor.kicad_sch
- sheet USB: file schematics/USB-C.kicad_sch -> schematics/usb_condor.kicad_sch
- note added: "Interfaces"
- note added: "Sensors"
- company: (none) -> Avionics @ Carnegie Mellon Rocket Command

Commit message: added rf schematic
Other:
- added sheet RF (schematics/rf_condor.kicad_sch)
Changed lines of the file:
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@@
 	(rectangle
 		(start 213.36 25.4)
-		(end 271.78 148.59)
+		(end 271.78 154.94)
 		(stroke
 			(width 0)
@@
 	(sheet
 		(at 217.17 34.29)
-		(size 50.8 50.8)
+		(size 50.8 31.75)
 		(exclude_from_sim no)
 		(in_bom yes)
@@
 		)
 		(property "Sheetfile" "schematics/usb_condor.kicad_sch"
-			(at 217.17 85.6746 0)
+			(at 217.17 66.6246 0)
 			(show_name no)
 			(do_not_autoplace no)
@@
 	)
 	(sheet
-		(at 217.17 92.71)
-		(size 50.8 50.8)
+		(at 217.17 76.2)
+		(size 50.8 31.75)
 		(exclude_from_sim no)
 		(in_bom yes)
@@
 		)
 		(property "Sheetname" "Storage"
-			(at 217.17 91.9984 0)
+			(at 217.17 75.4884 0)
 			(show_name no)
 			(do_not_autoplace no)
@@
 		)
 		(property "Sheetfile" "schematics/storage_condor.kicad_sch"
-			(at 217.17 144.0946 0)
+			(at 217.17 108.5346 0)
 			(show_name no)
 			(do_not_autoplace no)
@@
 				)
 			)
+		)
+	)
+	(sheet
+		(at 217.17 118.11)
+		(size 50.8 31.75)
+		(exclude_from_sim no)
+		(in_bom yes)
+		(on_board yes)
+		(dnp no)
+		(fields_autoplaced yes)
+		(stroke
+			(width 0.1524)
+			(type solid)
+		)
+		(fill
+			(color 255 153 0 0.25)
+		)
+		(property "Sheetname" "RF"
+			(at 217.17 117.3984 0)
+			(show_name no)
+			(do_not_autoplace no)
+			(effects
+				(font
+					(size 1.27 1.27)
+				)
+				(justify left bottom)
+			)
+		)
+		(property "Sheetfile" "schematics/rf_condor.kicad_sch"
+			(at 217.17 150.4446 0)
+			(show_name no)
+			(do_not_autoplace no)
+			(effects
+				(font
+					(size 1.27 1.27)
+				)
+				(justify left top)
+			)
+		)
+		(instances
+			(project "condor"
+				(path "/4a4947c5-540a-4852-b2fa-01bf36e5263c"
+					(page "13")
+				)
+			)
