File: schematics/Power.kicad_sch (KiCad schematic)
At the start: 20 parts, among them IC2 TPS563209DDCR, U5 IC MCU 32BIT 1MB FLASH 64LQFP

Commit message: Reorganizing + importing a few symbols
Parts:
- removed U5: IC MCU 32BIT 1MB FLASH 64LQFP, LQFP64-10x10mm, symbol Misc:STM32F4xxR2_minimalist
- added U2: STM32F413RGT6, LQFP64-10x10mm, symbol Condor_Imported_Symbols:STM32F413RGT6
Connections:
- net GND: now also U2.12 (VSSA/VREF-), U2.18 (VSS), U2.31 (VSS), U2.47 (VSS), U2.63 (VSS)
- net VCC_3V3: now also U2.1 (VBAT), U2.13 (VDDA/VREF+), U2.19 (VDD), U2.32 (VDD), U2.48 (VDD), U2.64 (VDD)
- net at C3.2: now also U2.30 (VCAP_1)
Other:
- note added: "TODO: Switch out MCU to whatever we decide on Verify this works Probably move the MCU power/decoupling into MCU file or MCU Power file Resolve imports: may need to swap to KiCad symbols"
- note removed: "TODO: Switch out MCU to whatever we decide on Verify this works Probably move the MCU power/decoupling into MCU file or MCU Power file Resolve imports"
