File: schematics/USB-C.kicad_sch (KiCad schematic)
At the start: 3 parts, among them J3 CX90M-16P

Commit message: Reorganizing + importing a few symbols
Other:
- note added: "Stolen from Kingfisher Symbol from Altium. May need to replace"
- note removed: "Stolen from Kingfisher Fix imports"
Changed lines of the file:
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@@
 	(generator_version "10.0")
 	(paper "A4")
-	(text "Stolen from Kingfisher\n\nFix imports"
+	(text "Stolen from Kingfisher\n\nSymbol from Altium. May need to replace"
 		(exclude_from_sim no)
 		(at 25.4 179.07 0)
