File: schematics/mcu_condor.kicad_sch (KiCad schematic)
At the start: 1 part, among them U2 STM32F413RGT6

Commit message: Update kicad_pro and kicad_sch + starting MCU
Parts:
- added LED1: LTST-C193KGKT-5A, LED_LTST-C193KGKT-5A:LED_LTST-C193KGKT-5A, symbol LED_LTST-C193KGKT-5A:LTST-C193KGKT-5A
- added LED2: LTST-C193KRKT-5A, LED_LTST-C193KRKT-5A:LED_LTST-C193KRKT-5A, symbol LED_LTST-C193KRKT-5A:LTST-C193KRKT-5A
Connections:
- net UART4_TX: now reaches U2.14 (PA0)
- net UART4_RX: now reaches U2.15 (PA1)
- net USART2_TX: now reaches U2.16 (PA2)
- net USART2_RX: now reaches U2.17 (PA3)
- net SPI2_CS: now reaches U2.33 (PB12)
- net SPI2_SCK: now reaches U2.34 (PB13)
- net SPI2_MOSI: now reaches U2.35 (PB14)
- net SPI2_MISO: now reaches U2.36 (PB15)
- net SPI3_SCK: now reaches U2.51 (PC10)
- net SPI3_MISO: now reaches U2.52 (PC11)
- net SPI3_MOSI: now reaches U2.53 (PC12)
- net SPI3_CS: now reaches U2.54 (PD2)
- net SPI1_SCK: now reaches U2.55 (PB3)
- net SPI1_MISO: now reaches U2.56 (PB4)
- net SPI1_MOSI: now reaches U2.57 (PB5)
- net SPI1_CS: now reaches U2.58 (PB6)
- net UART5: now reaches U2.61 (PB8)
Other:
- note added: "Cs set to NSS pin, which has predefined behavior. Switch to GPIO?"
- note added: "TODO: Oscillator, boot, USB, storage. RF and GPS are UART/USART? Likely need testpoints for debugging + status LEDS"
- note added: "What LEDS do I need? Power Safety Pyros MCU Maybe GPS and whatnot"

Commit message: Initial commit
Parts:
- removed LED2: LTST-C193KRKT-5A, LED_LTST-C193KRKT-5A:LED_LTST-C193KRKT-5A, symbol LED_LTST-C193KRKT-5A:LTST-C193KRKT-5A
- added LED_GPS: LTST-C193KGKT-5A, LED_LTST-C193KGKT-5A:LED_LTST-C193KGKT-5A, symbol LED_LTST-C193KGKT-5A:LTST-C193KGKT-5A
- added LED_MCU_STATUS, LED_PYRO, LED_RF_RX, LED_RF_TX: LTST-C193KRKT-5A, LED_LTST-C193KRKT-5A:LED_LTST-C193KRKT-5A, symbol LED_LTST-C193KRKT-5A:LTST-C193KRKT-5A
- renumbered LED1 to LED_POWER
Connections:
- net SPI3_CS: now also U2.50 (PA15); no longer U2.54 (PD2)
- net SPI1_CS2: now reaches U2.59 (PB7)
- net UART5_2?: now reaches U2.62 (PB9)
- net SPI1_CS renamed SPI1_CS1
- net UART5 renamed UART5_?
- new net SPI1_CS3: U2.54 (PD2)
- no-connect marks 0 -> 28
Other:
- note added: "Add interrupts"
- note added: "Need more CS"
