File: schematics/gps_condor.kicad_sch (KiCad schematic)
At the start: 0 parts

Commit message: Adding GNSS receiver symbols/footprint
Imported GNSS receiver footprints/symbols and added the symbol to the schematic
Parts:
- added U3: MAX-M10M-00B, MOD18_MAX-M10M_UBL, symbol MAX-M10N-10B:MAX-M10M-00B
Connections:
- new net GND: U3.1 (GND)
- new net {GPS_UART}: U3.2 (TXD), U3.3 (RXD)
